File: PCB/PiicoDev-Radio.kicad_sch (KiCad schematic)
At the start: 22 parts, among them J1 , J2 , J3 Conn_01x05_Male, SW1 ADDR, U1 ATtiny1616-M

Commit message: Update
Parts:
- added C2: 100n, Capacitor_SMD:C_0402_1005Metric, symbol Device:C
- added J4: Conn_Coaxial, Connector_Coaxial:SMB_Jack_Vertical, symbol Connector:Conn_Coaxial
- added U2: RFM69HCW, RF_Module:HOPERF_RFM9XW_SMD, symbol RF_Module:RFM69HCW
Connections:
- net +3V3: now also C2.2
- net GND: now also C2.1, J4.2 (Ext), U2.1 (GND), U2.10 (GND), U2.8 (GND)
- new net RF: J4.1 (In), U2.9 (ANT)
Changed lines of the file:
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@@
   (junction (at 63.5 157.48) (diameter 0) (color 0 0 0 0)
+  )
+  (junction (at 167.64 119.38) (diameter 0) (color 0 0 0 0)
   )
   (junction (at 63.5 154.94) (diameter 0) (color 0 0 0 0)
@@
     (stroke (width 0) (type default) (color 0 0 0 0))
   )
+  (wire (pts (xy 167.64 119.38) (xy 167.64 120.65))
+    (stroke (width 0) (type default) (color 0 0 0 0))
+  )
   (wire (pts (xy 67.31 107.95) (xy 67.31 120.65))
     (stroke (width 0) (type default) (color 0 0 0 0))
   )
+  (wire (pts (xy 170.18 119.38) (xy 170.18 118.11))
+    (stroke (width 0) (type default) (color 0 0 0 0))
+  )
   (wire (pts (xy 45.72 157.48) (xy 46.99 157.48))
     (stroke (width 0) (type default) (color 0 0 0 0))
   )
+  (wire (pts (xy 167.64 119.38) (xy 170.18 119.38))
+    (stroke (width 0) (type default) (color 0 0 0 0))
+  )
   (polyline (pts (xy 133.35 196.85) (xy 133.35 182.88))
     (stroke (width 0) (type default) (color 0 0 0 0))
@@
     (stroke (width 0) (type default) (color 0 0 0 0))
   )
+  (wire (pts (xy 201.93 100.33) (xy 201.93 114.3))
+    (stroke (width 0) (type default) (color 0 0 0 0))
+  )
   (polyline (pts (xy 63.5 127) (xy 100.33 127))
     (stroke (width 0) (type default) (color 0 0 0 0))
@@
     (stroke (width 0) (type default) (color 0 0 0 0))
   )
+  (wire (pts (xy 180.34 95.25) (xy 196.85 95.25))
+    (stroke (width 0) (type default) (color 0 0 0 0))
+  )
+  (wire (pts (xy 165.1 118.11) (xy 165.1 119.38))
+    (stroke (width 0) (type default) (color 0 0 0 0))
+  )
   (wire (pts (xy 219.71 85.09) (xy 219.71 81.28))
     (stroke (width 0) (type default) (color 0 0 0 0))
@@
     (stroke (width 0) (type default) (color 0 0 0 0))
   )
+  (wire (pts (xy 167.64 118.11) (xy 167.64 119.38))
+    (stroke (width 0) (type default) (color 0 0 0 0))
+  )
   (polyline (pts (xy 63.5 127) (xy 63.5 76.2))
     (stroke (width 0) (type default) (color 0 0 0 0))
@@
   )
   (wire (pts (xy 234.95 40.64) (xy 238.76 40.64))
+    (stroke (width 0) (type default) (color 0 0 0 0))
+  )
+  (wire (pts (xy 165.1 119.38) (xy 167.64 119.38))
     (stroke (width 0) (type default) (color 0 0 0 0))
   )
@@
   )
   (label "SCL" (at 41.91 57.15 0)
+    (effects (font (size 1.27 1.27)) (justify left bottom))
+  )
+  (label "RF" (at 187.96 95.25 0)
     (effects (font (size 1.27 1.27)) (justify left bottom))
   )
@@
     )
   )
+  (symbol (lib_id "power:GND") (at 143.51 144.78 0) (unit 1)
+    (in_bom yes) (on_board yes)
+    (property "Reference" "#PWR0115" (id 0) (at 143.51 151.13 0)
+      (effects (font (size 1.27 1.27)) hide)
+    )
+    (property "Value" "GND" (id 1) (at 143.637 148.0312 90)
+      (effects (font (size 1.27 1.27)) (justify right))
+    )
+    (property "Footprint" "" (id 2) (at 143.51 144.78 0)
+      (effects (font (size 1.27 1.27)) hide)
+    )
+    (property "Datasheet" "" (id 3) (at 143.51 144.78 0)
+      (effects (font (size 1.27 1.27)) hide)
+    )
+    (pin "1")
+  )
   (symbol (lib_id "Mechanical:MountingHole") (at 161.925 186.69 0) (unit 1)
     (in_bom yes) (on_board yes)
@@
     (pin "5")
   )
+  (symbol (lib_id "Connector:Conn_Coaxial") (at 201.93 95.25 0) (unit 1)
+    (in_bom yes) (on_board yes) (fields_autoplaced)
+    (property "Reference" "J4" (id 0) (at 204.47 94.2731 0)
+      (effects (font (size 1.27 1.27)) (justify left))
+    )
+    (property "Value" "Conn_Coaxial" (id 1) (at 204.47 96.8131 0)
+      (effects (font (size 1.27 1.27)) (justify left))
+    )
+    (property "Footprint" "Connector_Coaxial:SMB_Jack_Vertical" (id 2) (at 201.93 95.25 0)
+      (effects (font (size 1.27 1.27)) hide)
+    )
+    (property "Datasheet" " ~" (id 3) (at 201.93 95.25 0)
+      (effects (font (size 1.27 1.27)) hide)
+    )
+    (pin "1")
+    (pin "2")
+  )
   (symbol (lib_id "Device:R") (at 240.03 66.04 90) (unit 1)
     (in_bom yes) (on_board yes)
@@
     (pin "2")
   )
+  (symbol (lib_id "RF_Module:RFM69HCW") (at 167.64 102.87 0) (unit 1)
+    (in_bom yes) (on_board yes) (fields_autoplaced)
+    (property "Reference" "U2" (id 0) (at 169.6594 87.63 0)
+      (effects (font (size 1.27 1.27)) (justify left))
+    )
+    (property "Value" "RFM69HCW" (id 1) (at 169.6594 90.17 0)
+      (effects (font (size 1.27 1.27)) (justify left))
+    )
+    (property "Footprint" "RF_Module:HOPERF_RFM9XW_SMD" (id 2) (at 83.82 60.96 0)
+      (effects (font (size 1.27 1.27)) hide)
+    )
+    (property "Datasheet" "https://www.hoperf.com/data/upload/portal/20181127/5bfcb8284d838.pdf" (id 3) (at 83.82 60.96 0)
+      (effects (font (size 1.27 1.27)) hide)
+    )
+    (pin "1")
+    (pin "10")
+    (pin "11")
+    (pin "12")
+    (pin "13")
+    (pin "14")
+    (pin "15")
+    (pin "16")
+    (pin "2")
+    (pin "3")
+    (pin "4")
+    (pin "5")
+    (pin "6")
+    (pin "7")
+    (pin "8")
+    (pin "9")
+  )
+  (symbol (lib_id "power:GND") (at 167.64 120.65 0) (unit 1)
+    (in_bom yes) (on_board yes) (fields_autoplaced)
+    (property "Reference" "#PWR0119" (id 0) (at 167.64 127 0)
+      (effects (font (size 1.27 1.27)) hide)
+    )
+    (property "Value" "GND" (id 1) (at 167.64 125.73 0))
+    (property "Footprint" "" (id 2) (at 167.64 120.65 0)
+      (effects (font (size 1.27 1.27)) hide)
+    )
+    (property "Datasheet" "" (id 3) (at 167.64 120.65 0)
+      (effects (font (size 1.27 1.27)) hide)
+    )
+    (pin "1")
+  )
   (symbol (lib_id "power:GND") (at 88.9 38.1 90) (unit 1)
     (in_bom yes) (on_board yes)
@@
     (pin "1")
   )
+  (symbol (lib_id "power:+3V3") (at 143.51 137.16 0) (unit 1)
+    (in_bom yes) (on_board yes)
+    (property "Reference" "#PWR0114" (id 0) (at 143.51 140.97 0)
+      (effects (font (size 1.27 1.27)) hide)
+    )
+    (property "Value" "+3V3" (id 1) (at 143.891 132.7658 0))
+    (property "Footprint" "" (id 2) (at 143.51 137.16 0)
+      (effects (font (size 1.27 1.27)) hide)
+    )
+    (property "Datasheet" "" (id 3) (at 143.51 137.16 0)
+      (effects (font (size 1.27 1.27)) hide)
+    )
+    (pin "1")
+  )
+  (symbol (lib_id "Device:C") (at 143.51 140.97 0) (mirror x) (unit 1)
+    (in_bom yes) (on_board yes)
+    (property "Reference" "C2" (id 0) (at 146.431 142.1384 0)
+      (effects (font (size 1.27 1.27)) (justify left))
+    )
+    (property "Value" "100n" (id 1) (at 146.431 139.827 0)
+      (effects (font (size 1.27 1.27)) (justify left))
+    )
+    (property "Footprint" "Capacitor_SMD:C_0402_1005Metric" (id 2) (at 144.4752 137.16 0)
+      (effects (font (size 1.27 1.27)) hide)
+    )
+    (property "Datasheet" "~" (id 3) (at 143.51 140.97 0)
+      (effects (font (size 1.27 1.27)) hide)
+    )
+    (pin "1")
+    (pin "2")
+  )
   (symbol (lib_id "power:+3V3") (at 88.9 40.64 270) (unit 1)
     (in_bom yes) (on_board yes)
@@
     )
     (property "Datasheet" "" (id 3) (at 88.9 40.64 0)
+      (effects (font (size 1.27 1.27)) hide)
+    )
+    (pin "1")
+  )
+  (symbol (lib_id "power:GND") (at 201.93 114.3 0) (unit 1)
+    (in_bom yes) (on_board yes) (fields_autoplaced)
+    (property "Reference" "#PWR0118" (id 0) (at 201.93 120.65 0)
+      (effects (font (size 1.27 1.27)) hide)
+    )
+    (property "Value" "GND" (id 1) (at 201.93 119.38 0))
+    (property "Footprint" "" (id 2) (at 201.93 114.3 0)
+      (effects (font (size 1.27 1.27)) hide)
+    )
+    (property "Datasheet" "" (id 3) (at 201.93 114.3 0)
       (effects (font (size 1.27 1.27)) hide)
     )
@@
       (reference "#PWR0113") (unit 1) (value "+3V3") (footprint "")
     )
+    (path "/bb51b2b2-a66b-48b5-8b1c-ceb898fbb6f7"
+      (reference "#PWR0114") (unit 1) (value "+3V3") (footprint "")
+    )
+    (path "/45c58424-ee39-46b5-8cc4-592fad2d7711"
+      (reference "#PWR0115") (unit 1) (value "GND") (footprint "")
+    )
     (path "/ba55cec1-41fe-4c9a-9957-8c8c51f2e64e"
       (reference "#PWR0116") (unit 1) (value "GND") (footprint "")
@@
       (reference "#PWR0117") (unit 1) (value "+3V3") (footprint "")
     )
+    (path "/d6b6c976-d855-4e1c-8189-4a70d45ef7e6"
+      (reference "#PWR0118") (unit 1) (value "GND") (footprint "")
+    )
+    (path "/a371a2d9-ae21-451d-9ace-05265aa9b4c3"
+      (reference "#PWR0119") (unit 1) (value "GND") (footprint "")
+    )
     (path "/00000000-0000-0000-0000-000061308deb"
       (reference "C1") (unit 1) (value "100n") (footprint "Capacitor_SMD:C_0402_1005Metric")
     )
+    (path "/c6625604-599a-4f2a-8cc6-c370e9c870af"
+      (reference "C2") (unit 1) (value "100n") (footprint "Capacitor_SMD:C_0402_1005Metric")
+    )
     (path "/00000000-0000-0000-0000-000060a1f602"
       (reference "D1") (unit 1) (value "LED") (footprint "LED_SMD:LED_0603_1608Metric")
@@
       (reference "J3") (unit 1) (value "Conn_01x05_Male") (footprint "CoreElectronics_Components:TestPoint_Pad_D1.0mm_x05_Pattern1")
     )
+    (path "/716e0700-d216-4aea-bb7d-f7a2fdc8ea94"
+      (reference "J4") (unit 1) (value "Conn_Coaxial") (footprint "Connector_Coaxial:SMB_Jack_Vertical")
+    )
     (path "/00000000-0000-0000-0000-000060a08168"
       (reference "JP2") (unit 1) (value "I2C PU") (footprint "CoreElectronics_Components:SolderJumper-3_P1.3mm_Closed_RoundedPad1.0x1.5mm_NumberLabels")
@@
       (reference "U1") (unit 1) (value "ATtiny1616-M") (footprint "Package_DFN_QFN:VQFN-20-1EP_3x3mm_P0.4mm_EP1.7x1.7mm")
     )
-  )
+    (path "/9f2b6969-af43-4436-9467-21310d788367"
+      (reference "U2") (unit 1) (value "RFM69HCW") (footprint "RF_Module:HOPERF_RFM9XW_SMD")
+    )
+  )

Commit message: Basic design complete
Parts:
- added C3: 100u, Capacitor_SMD:C_0603_1608Metric, symbol Device:C
- added D2: LED, LED_SMD:LED_0603_1608Metric, symbol Device:LED
- added JP1: SolderJumper_2_Bridged, CoreElectronics_Components:SolderJumper-2_P1.3mm_Bridged_RoundedPad1.0x1.5mm, symbol Jumper:SolderJumper_2_Bridged
- added R5: 510R, Resistor_SMD:R_0402_1005Metric, symbol Device:R
Connections:
- net +3V3: now also U2.13 (3.3V), C3.2
- net ADD1: now also U1.18 (PC3); no longer U1.20 (PA1)
- net ADD2: now also U1.17 (PC2); no longer U1.18 (PC3)
- net ADD3: now also U1.16 (PC1); no longer U1.17 (PC2)
- net ADD4: now also U1.15 (PC0); no longer U1.16 (PC1)
- net GND: now also C3.1, D2.1 (K)
- net PWR_LED: now also U1.6 (PA5); no longer U1.2 (PA3)
- net MISO: now reaches U1.1 (PA2)
- net MISO: now also U2.2 (MISO)
- net DIO0: now reaches U1.10 (PB4)
- net DIO0: now also U2.14 (DIO0), JP1.2 (B)
- net DIO4: now reaches U1.11 (PB3)
- net DIO4: now also U2.12 (DIO4)
- net DIO3: now reaches U1.12 (PB2)
- net DIO3: now also U2.11 (DIO3)
- net NSS: now reaches U1.5 (PA4)
- net NSS: now also U2.5 (NSS)
- net RESET: now reaches U1.7 (PA6)
- net RESET: now also U2.6 (RESET)
- net DIO2: now reaches U1.8 (PA7)
- net DIO2: now also U2.16 (DIO2)
- net DIO1: now reaches U1.9 (PB5)
- net DIO1: now also U2.15 (DIO1)
- net MOSI: now reaches U2.3 (MOSI)
- net MOSI: now also U1.20 (PA1)
- net SCK: now reaches U2.4 (SCK)
- net SCK: now also U1.2 (PA3)
- new net: D2.2 (A), R5.2
- new net: JP1.1 (A), R5.1
- no-connect marks 10 -> 1
Other:
- note added: "LED Vf = 2.8 V RFM69HCW DIO Maximum Current = 1 mA R = (3.3 - 2.8)/0.001 = 500 Ohms"
- note added: "Rx: CrcOk Tx: PacketSent"
- moved on the sheet: C1, C2, J4, R4, U1, U2

Commit message: Remove SMA and add PCB antenna
Parts:
- removed H4: MountingHole, CoreElectronics_Components:MountingHole_2.7mm_M2.5_PadClearance_1.2, symbol Mechanical:MountingHole
- removed J4: Conn_Coaxial, Connector_Coaxial:SMB_Jack_Vertical, symbol Connector:Conn_Coaxial
- added AE1: Antenna_Chip_No_Antenna_Symbol, CoreElectronics_Components:Antenna_Chip_TDK_ANT160920ST-1204A1, symbol Project Library:Antenna_Chip_No_Antenna_Symbol
- added AE2: Antenna, Project Library:PiicoDev_Radio_Antenna, symbol Device:Antenna
- added L1, L2, L3: L, Inductor_SMD:L_0402_1005Metric, symbol Device:L
- C3: value 100u -> 10u
Connections:
- net GND: now also L1.1
- net RF: now also L1.2, L2.1
- new net: AE1.1 (PCB_Trace), AE2.1 (A)
- new net RF1: L2.2, L3.1
- new net RF2: AE1.4 (FEED), L3.2

Commit message: update
Parts:
- FID1, FID2, G1, G2, G3, H1, H2, H3, J3, JP1, JP2, LOGO1: now left out of the parts list
Changed lines of the file:
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@@
     (stroke (width 0) (type solid) (color 0 0 0 0))
+  )
+  (polyline (pts (xy 246.38 40.64) (xy 246.38 44.45))
+    (stroke (width 0) (type default) (color 0 0 0 0))
   )
   (wire (pts (xy 179.07 39.37) (xy 186.69 39.37))
@@
     (stroke (width 0) (type default) (color 0 0 0 0))
   )
+  (polyline (pts (xy 256.54 44.45) (xy 256.54 48.26))
+    (stroke (width 0) (type default) (color 0 0 0 0))
+  )
   (polyline (pts (xy 175.26 196.85) (xy 166.37 196.85))
     (stroke (width 0) (type default) (color 0 0 0 0))
@@
   )
   (wire (pts (xy 166.37 52.07) (xy 167.64 52.07))
+    (stroke (width 0) (type default) (color 0 0 0 0))
+  )
+  (polyline (pts (xy 256.54 48.26) (xy 267.97 48.26))
     (stroke (width 0) (type default) (color 0 0 0 0))
   )
@@
     (stroke (width 0) (type solid) (color 0 0 0 0))
   )
+  (polyline (pts (xy 245.11 44.45) (xy 256.54 44.45))
+    (stroke (width 0) (type default) (color 0 0 0 0))
+  )
   (wire (pts (xy 41.91 57.15) (xy 36.83 57.15))
     (stroke (width 0) (type default) (color 0 0 0 0))
@@
     (stroke (width 0) (type default) (color 0 0 0 0))
   )
+  (polyline (pts (xy 254 40.64) (xy 254 44.45))
+    (stroke (width 0) (type default) (color 0 0 0 0))
+  )
   (polyline (pts (xy 25.4 127) (xy 62.23 127))
     (stroke (width 0) (type default) (color 0 0 0 0))
@@
   )
   (symbol (lib_id "CoreElectronics_Artwork:LOGO_PiicoDev") (at 203.2 160.02 0) (unit 1)
-    (in_bom yes) (on_board yes)
+    (in_bom no) (on_board yes)
     (property "Reference" "G1" (id 0) (at 203.2 165.7096 0)
       (effects (font (size 1.524 1.524)) hide)
@@
   )
   (symbol (lib_id "CoreElectronics_Artwork:LOGO_made-with-love") (at 269.24 158.75 0) (unit 1)
-    (in_bom yes) (on_board yes)
+    (in_bom no) (on_board yes)
     (property "Reference" "G3" (id 0) (at 269.24 163.9824 0)
       (effects (font (size 1.524 1.524)) hide)
@@
   )
   (symbol (lib_id "CoreElectronics_Artwork:LOGO_CoreElectronics_no-text") (at 251.46 158.75 0) (unit 1)
-    (in_bom yes) (on_board yes)
+    (in_bom no) (on_board yes)
     (property "Reference" "G2" (id 0) (at 251.46 163.9824 0)
       (effects (font (size 1.524 1.524)) hide)
@@
   )
   (symbol (lib_id "Graphic:Logo_Open_Hardware_Small") (at 276.86 173.99 0) (unit 1)
-    (in_bom yes) (on_board yes)
+    (in_bom no) (on_board yes)
     (property "Reference" "LOGO1" (id 0) (at 276.86 167.005 0)
       (effects (font (size 1.27 1.27)) hide)
@@
   )
   (symbol (lib_id "Mechanical:MountingHole") (at 157.48 191.77 0) (unit 1)
-    (in_bom yes) (on_board yes)
+    (in_bom no) (on_board yes)
     (property "Reference" "H2" (id 0) (at 160.02 190.6016 0)
       (effects (font (size 1.27 1.27)) (justify left) hide)
@@
   )
   (symbol (lib_id "Mechanical:MountingHole") (at 157.48 186.69 0) (unit 1)
-    (in_bom yes) (on_board yes)
+    (in_bom no) (on_board yes)
     (property "Reference" "H1" (id 0) (at 160.02 185.5216 0)
       (effects (font (size 1.27 1.27)) (justify left) hide)
@@
   )
   (symbol (lib_id "Mechanical:Fiducial") (at 170.18 190.5 0) (unit 1)
-    (in_bom yes) (on_board yes)
+    (in_bom no) (on_board yes)
     (property "Reference" "FID2" (id 0) (at 172.339 189.3316 0)
       (effects (font (size 1.27 1.27)) (justify left) hide)
@@
   )
   (symbol (lib_id "Mechanical:Fiducial") (at 170.18 186.69 0) (unit 1)
-    (in_bom yes) (on_board yes)
+    (in_bom no) (on_board yes)
     (property "Reference" "FID1" (id 0) (at 172.339 185.5216 0)
       (effects (font (size 1.27 1.27)) (justify left) hide)
@@
   )
   (symbol (lib_id "Jumper:SolderJumper_3_Bridged123") (at 74.93 92.71 180) (unit 1)
-    (in_bom yes) (on_board yes)
+    (in_bom no) (on_board yes)
     (property "Reference" "JP2" (id 0) (at 74.93 95.5802 0))
     (property "Value" "I2C PU" (id 1) (at 74.93 97.8916 0))
@@
   )
   (symbol (lib_id "Mechanical:MountingHole") (at 161.925 186.69 0) (unit 1)
-    (in_bom yes) (on_board yes)
+    (in_bom no) (on_board yes)
     (property "Reference" "H3" (id 0) (at 164.465 185.5216 0)
       (effects (font (size 1.27 1.27)) (justify left) hide)
@@
   )
   (symbol (lib_id "Connector:Conn_01x05_Male") (at 74.93 43.18 0) (unit 1)
-    (in_bom yes) (on_board yes) (fields_autoplaced)
+    (in_bom no) (on_board yes) (fields_autoplaced)
     (property "Reference" "J3" (id 0) (at 75.565 35.56 0))
     (property "Value" "Conn_01x05_Male" (id 1) (at 75.565 40.64 0)
@@
   )
   (symbol (lib_id "Jumper:SolderJumper_2_Bridged") (at 222.25 57.15 180) (unit 1)
-    (in_bom yes) (on_board yes)
+    (in_bom no) (on_board yes)
     (property "Reference" "JP1" (id 0) (at 220.9799 54.61 90)
       (effects (font (size 1.27 1.27)) (justify right))

Commit message: Change R5 to 1k
Parts:
- R5: value 510R -> 1k
Other:
- note added: "LED Vf = 2.8 V RFM69HCW DIO Maximum Current = 1 mA R = (3.3 - 2.8)/0.001 = 500 Ohms Round to 1k to use more common part"
- note removed: "LED Vf = 2.8 V RFM69HCW DIO Maximum Current = 1 mA R = (3.3 - 2.8)/0.001 = 500 Ohms"
Changed lines of the file:
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@@
     (effects (font (size 1.27 1.27)) (justify left bottom))
   )
-  (text "LED Vf = 2.8 V\nRFM69HCW DIO Maximum Current = 1 mA\nR = (3.3 - 2.8)/0.001 = 500 Ohms"
+  (text "LED Vf = 2.8 V\nRFM69HCW DIO Maximum Current = 1 mA\nR = (3.3 - 2.8)/0.001 = 500 Ohms\nRound to 1k to use more common part"
     (at 210.82 97.79 0)
     (effects (font (size 1.27 1.27)) (justify left bottom))
@@
       (effects (font (size 1.27 1.27)) (justify left))
     )
-    (property "Value" "510R" (id 1) (at 233.68 59.69 90)
+    (property "Value" "1k" (id 1) (at 233.68 59.69 90)
       (effects (font (size 1.27 1.27)) (justify left))
     )
@@
     )
     (path "/b1580650-e108-427e-8f52-7d58a58420ac"
-      (reference "R5") (unit 1) (value "510R") (footprint "Resistor_SMD:R_0402_1005Metric")
+      (reference "R5") (unit 1) (value "1k") (footprint "Resistor_SMD:R_0402_1005Metric")
     )
     (path "/00000000-0000-0000-0000-00006138b025"
